File: Hardware/Qwiic EEPROM.sch (EAGLE design)
At the start: 29 parts, among them J2 SMD, J3 PTH, J4 SMD, U1 RM24C512C

Commit message: added address chart to schematic
Other:
- note added: "0x50"
- note added: "0x51"
- note added: "0x52"
- note added: "0x53"
- note added: "0x54"
- note added: "0x55"
- note added: "0x56"
- note added: "0x57"
- note added: "ADDRESS"
- note added: "E0"
- note added: "E1"
- note added: "E2"
- moved on the sheet: C4, D1, E0, E1, E2, I2C, J1, R1, R2, R3, R4, R5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

Commit message: documentation
Parts:
- J2, J4: value SMD -> (none); device SparkX:I2C_STANDARDJS-1MM -> SparkFun-Connectors:QWIIC_CONNECTORJS-1MM
Connections:
- net 3.3V: now also J2.2, J4.2; no longer J2.VCC, J4.VCC
- net GND: now also J2.1, J4.1; no longer J2.GND, J4.GND
- net SCL: now also J2.4, J4.4; no longer J2.SCL, J4.SCL
- net SDA: now also J2.3, J4.3; no longer J2.SDA, J4.SDA
Other:
- moved on the sheet: C4, D1, E0, E1, E2, I2C, J1, J2, J3, J4, R1, R2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
